File: KiCadProject/079721-2351/079721-2351.kicad_pcb (KiCad board)
At the start: 2 copper layers, 25 parts, among them J1 Mazda_02x11, J2 Conn_02x13_Odd_Even, J711 Empty, T822 empty, T831 Empty, T832 Empty, T851 Empty, T852 empty, T861 Empty

Commit message: elements1
Parts:
- added C1: 47nf, ProjektMazda:capacitorTantalumMazda6mm, F.Cu at (123.9, -19.1)
- added C105: 47nf, ProjektMazda:capacitorTantalumMazda6mm, F.Cu at (132.5, -15.8)
- added C205: 47nf, ProjektMazda:capacitorTantalumMazda6mm, F.Cu at (123.9, -9.35)
- added C3: 47nf, ProjektMazda:capacitorTantalumMazda6mm, F.Cu at (132.5, -19.1)
- added C401: 10nF (103), ProjektMazda:capacitorTantalumMazda6mm, F.Cu at (196.3, -20.2)
- added C405: 10nF (103), ProjektMazda:capacitorTantalumMazda6mm, F.Cu at (179.1, -7.20)
- added C421: 47nf, ProjektMazda:capacitorTantalumMazda6mm, F.Cu at (63.6, -23.4)
- added C422: 10nF (103), ProjektMazda:capacitorTantalumMazda6mm, F.Cu at (196.3, -16.9)
- added C431: 47nf, ProjektMazda:capacitorTantalumMazda6mm, F.Cu at (63.6, -20.2)
- added C432: 10nF (103), ProjektMazda:capacitorTantalumMazda6mm, F.Cu at (179.1, -20.2)
- added C441: empty, ProjektMazda:capacitorTantalumMazda6mm, F.Cu at (63.6, -16.9)
- added C442: 10nF (103), ProjektMazda:capacitorTantalumMazda6mm, F.Cu at (187.7, -10.4)
- added C451: 47nf, ProjektMazda:capacitorTantalumMazda6mm, F.Cu at (123.9, -15.8)
- added C452: 47nf, ProjektMazda:capacitorTantalumMazda6mm, F.Cu at (141.1, -19.1)
- added C461: 10nF (103), ProjektMazda:capacitorTantalumMazda6mm, F.Cu at (179.1, -3.95)
- added C471: 47nf, ProjektMazda:capacitorTantalumMazda6mm, F.Cu at (123.9, -12.6)
- added C472: 10nF (103), ProjektMazda:capacitorTantalumMazda6mm, F.Cu at (204.9, -20.2)
- added C481: 10nF (103), ProjektMazda:capacitorTantalumMazda6mm, F.Cu at (187.7, -7.20)
- added C491: 10nF (103), ProjektMazda:capacitorTantalumMazda6mm, F.Cu at (196.3, -13.7)
- added C5: 10nF (103), ProjektMazda:capacitorTantalumMazda6mm, F.Cu at (187.7, -13.7)
- added C503: 47nf, ProjektMazda:capacitorTantalumMazda6mm, F.Cu at (132.5, -12.6)
- added C504: 47nf, ProjektMazda:capacitorTantalumMazda6mm, F.Cu at (141.1, -15.8)
- added C511: 47nf, ProjektMazda:capacitorTantalumMazda6mm, F.Cu at (132.5, -9.35)
- added C52: 10nF (103), ProjektMazda:capacitorTantalumMazda6mm, F.Cu at (187.7, -20.2)
- added C54: 10nF (103), ProjektMazda:capacitorTantalumMazda6mm, F.Cu at (179.1, -13.7)
- added C55: 10nF (103), ProjektMazda:capacitorTantalumMazda6mm, F.Cu at (187.7, -16.9)
- added C56: 10nF (103), ProjektMazda:capacitorTantalumMazda6mm, F.Cu at (179.1, -10.4)
- added C603: 10nF (103), ProjektMazda:capacitorTantalumMazda6mm, F.Cu at (204.9, -16.9)
- added C607: 10nF (103), ProjektMazda:capacitorTantalumMazda6mm, F.Cu at (196.3, -10.4)
- added C9: 10nF (103), ProjektMazda:capacitorTantalumMazda6mm, F.Cu at (179.1, -16.9)
- added C911: 47nf, ProjektMazda:capacitorTantalumMazda6mm, F.Cu at (141.1, -12.6)
- added C921: 47nf, ProjektMazda:capacitorTantalumMazda6mm, F.Cu at (141.1, -9.35)
- added D1: 1E1, Diode_THT:DiodaMazda, F.Cu at (161.9, 84.0)
- added D3: 1E1, Diode_THT:DiodaMazda, F.Cu at (161.9, 87.3)
- added D4: 1E1, Diode_THT:DiodaMazda, F.Cu at (175.6, 84.0)
- added D801: 1E1, Diode_THT:DiodaMazda, F.Cu at (161.9, 90.6)
- added D802: 1E1, Diode_THT:DiodaMazda, F.Cu at (175.6, 87.3)
- added D811: 1E1, Diode_THT:DiodaMazda, F.Cu at (161.9, 93.9)
- added D812: 1E1, Diode_THT:DiodaMazda, F.Cu at (161.9, 97.2)
- added D851: empty, Diode_THT:DiodaMazda, F.Cu at (161.9, 100.5)
- added F401: 223s, murata-resonators:murata-resonators-CSTLS_G9, F.Cu at (101.0, 83.9)
- added R101: 1K, Resistor_THT:MazdaResistor10mm, F.Cu at (28.8, -30.3)
- added R102: 10k, Resistor_THT:MazdaResistor10mm, F.Cu at (79.2, -61.4)
- added R112: 10k, Resistor_THT:MazdaResistor10mm, F.Cu at (92.8, -64.2)
- added R2: 10k, Resistor_THT:MazdaResistor10mm, F.Cu at (79.2, -64.2)
- added R211: 10k, Resistor_THT:MazdaResistor10mm, F.Cu at (79.2, -58.6)
- added R402: 10k, Resistor_THT:MazdaResistor10mm, F.Cu at (92.8, -61.4)
- added R421: 2,7K2%, Resistor_THT:MazdaResistor10mm, F.Cu at (35.4, 0.60)
- added R422: 10k, Resistor_THT:MazdaResistor10mm, F.Cu at (79.2, -55.8)
- added R431: 2,7K2%, Resistor_THT:MazdaResistor10mm, F.Cu at (35.4, 3.40)
- added R441: 10k, Resistor_THT:MazdaResistor10mm, F.Cu at (79.2, -53.0)
- added R442: 10k, Resistor_THT:MazdaResistor10mm, F.Cu at (79.2, -50.2)
- added R451: empty, Resistor_THT:MazdaResistor10mm, F.Cu at (175.6, 90.3)
- added R461: empty, Resistor_THT:MazdaResistor10mm, F.Cu at (106.4, -64.2)
- added R463: 10k, Resistor_THT:MazdaResistor10mm, F.Cu at (35.4, 6.20)
- added R472: 10k, Resistor_THT:MazdaResistor10mm, F.Cu at (79.2, -47.4)
- added R481: 10k, Resistor_THT:MazdaResistor10mm, F.Cu at (92.8, -58.6)
- added R482: 10k, Resistor_THT:MazdaResistor10mm, F.Cu at (79.2, -44.6)
- added R491: empty, Resistor_THT:MazdaResistor10mm, F.Cu at (175.6, 93.1)
- added R492: empty, Resistor_THT:MazdaResistor10mm, F.Cu at (175.6, 95.9)
- added R501: 680R, ProjektMazda:MazdaResistor12mm, F.Cu at (137.2, -60.1)
- added R502: 2.2k, Resistor_THT:MazdaResistor10mm, F.Cu at (137.2, -46.1)
- added R503: 680R, ProjektMazda:MazdaResistor12mm, F.Cu at (152.0, -60.1)
- added R504: 2.2k, Resistor_THT:MazdaResistor10mm, F.Cu at (137.2, -43.3)
- added R505: 680R, ProjektMazda:MazdaResistor12mm, F.Cu at (152.0, -57.3)
- added R506: 2.2k, Resistor_THT:MazdaResistor10mm, F.Cu at (137.2, -40.5)
- added R507: 2.2k, Resistor_THT:MazdaResistor10mm, F.Cu at (150.8, -48.9)
- added R508: 2.2k, Resistor_THT:MazdaResistor10mm, F.Cu at (150.8, -46.1)
- added R509: empty, Resistor_THT:MazdaResistor10mm, F.Cu at (175.6, 98.7)
- added R510: 2.2k, Resistor_THT:MazdaResistor10mm, F.Cu at (164.4, -48.9)
- added R511: 10k, Resistor_THT:MazdaResistor10mm, F.Cu at (92.8, -55.8)
- added R512: 10k, Resistor_THT:MazdaResistor10mm, F.Cu at (106.4, -61.4)
- added R513: 10k, Resistor_THT:MazdaResistor10mm, F.Cu at (92.8, -53.0)
- added R514: 10k, Resistor_THT:MazdaResistor10mm, F.Cu at (28.8, -27.5)
- added R515: 10k, Resistor_THT:MazdaResistor10mm, F.Cu at (92.8, -50.2)
- added R516: 10k, Resistor_THT:MazdaResistor10mm, F.Cu at (92.8, -47.4)
- added R517: 10k, Resistor_THT:MazdaResistor10mm, F.Cu at (92.8, -44.6)
- added R518: 10k, Resistor_THT:MazdaResistor10mm, F.Cu at (106.4, -58.6)
- added R519: 10k, Resistor_THT:MazdaResistor10mm, F.Cu at (106.4, -55.8)
- added R521: 10k, Resistor_THT:MazdaResistor10mm, F.Cu at (106.4, -53.0)
- added R531: 680R, ProjektMazda:MazdaResistor12mm, F.Cu at (137.2, -51.7)
- added R532: 2.2k, Resistor_THT:MazdaResistor10mm, F.Cu at (152.0, -54.5)
- added R541: 10k, Resistor_THT:MazdaResistor10mm, F.Cu at (106.4, -50.2)
- added R542: 10k, Resistor_THT:MazdaResistor10mm, F.Cu at (106.4, -47.4)
- added R561: 10k, Resistor_THT:MazdaResistor10mm, F.Cu at (28.8, -24.7)
- added R722: 1k, Resistor_THT:MazdaResistor10mm, F.Cu at (106.4, -44.6)
- added R751: 2.2k, Resistor_THT:MazdaResistor10mm, F.Cu at (152.0, -51.7)
- added R753: 63R, ProjektMazda:MazdaResistor12mm, F.Cu at (137.2, -54.5)
- added R761: 2.2k, Resistor_THT:MazdaResistor10mm, F.Cu at (150.8, -43.3)
- added R763: 63R, ProjektMazda:MazdaResistor12mm, F.Cu at (137.2, -57.3)
- added R801: 2.2k, Resistor_THT:MazdaResistor10mm, F.Cu at (150.8, -40.5)
- added R805: 8.2R2W, ProjektMazda:R17mm, F.Cu at (35.4, -2.20)
- added R822: empty, ProjektMazda:R17mm, F.Cu at (108.4, 61.0)
- added R832: empty, ProjektMazda:R17mm, F.Cu at (108.4, 57.1)
- added R861: empty, Resistor_THT:MazdaResistor10mm, F.Cu at (137.2, -48.9)
- added c51: empty, ProjektMazda:capacitorTantalumMazda6mm, F.Cu at (167.3, -59.7)
- C111: value 10nF50V (103 50J NCC) -> 10nF50V
- C411: value 3.3Uf50Velectrolitic -> 3.3uf50Velec
- R806, R812: footprint ProjektMazda:MazdaResistor17mm -> ProjektMazda:R17mm
- moved R806 17.6 mm to (109.0, 53.5), turned to 180 degrees
- moved R813 9.06 mm to (99.2, 49.0)
- moved c861 7.60 mm to (96.5, 44.3), turned to 180 degrees
- renumbered C053 to C53
Routing:
- net Net-(J2-Pad2T): track 0.00 -> 68.9 mm
- net Net-(J2-Pad2Y): track 0.00 -> 27.9 mm
- net Net-(J2-Pad2W): track 0.00 -> 6.99 mm
- net Net-(J2-Pad2S): track 0.00 -> 5.93 mm

Commit message: Resistors
Parts:
- added C601: 20 pF (20), ProjektMazda:capacitorTantalumMazda6mm, F.Cu at (213.4, -41.2)
- added C602: 20 pF (20), ProjektMazda:capacitorTantalumMazda6mm, F.Cu at (213.4, -38.0)
- added C606: 20 pF (20), ProjektMazda:capacitorTantalumMazda6mm, F.Cu at (213.4, -34.7)
- added R104: 22k, Resistor_THT:MazdaResistor10mm, F.Cu at (24.7, -88.2)
- added R105: 13k, Resistor_THT:MazdaResistor10mm, F.Cu at (11.1, -82.6)
- added R106: 18k, Resistor_THT:MazdaResistor10mm, F.Cu at (199.3, -47.2)
- added R111: 1k, Resistor_THT:MazdaResistor10mm, F.Cu at (24.7, -85.4)
- added R114: 22k, Resistor_THT:MazdaResistor10mm, F.Cu at (11.1, -79.8)
- added R115: 13k, Resistor_THT:MazdaResistor10mm, F.Cu at (11.1, -77.0)
- added R116: 18k, Resistor_THT:MazdaResistor10mm, F.Cu at (199.3, -44.4)
- added R201: 68K 2%, Resistor_THT:MazdaResistor10mm, F.Cu at (212.9, -47.2)
- added R202: 100K 2%, Resistor_THT:MazdaResistor10mm, F.Cu at (199.3, -41.6)
- added R203: 68K 2%, Resistor_THT:MazdaResistor10mm, F.Cu at (212.9, -44.4)
- added R204: 36K 2%, Resistor_THT:MazdaResistor10mm, F.Cu at (199.3, -38.8)
- added R21: 22k, Resistor_THT:MazdaResistor10mm, F.Cu at (11.1, -85.4)
- added R401: 1.5M, Resistor_THT:MazdaResistor10mm, F.Cu at (11.1, -74.2)
- added R411: 1k 2%, Resistor_THT:MazdaResistor10mm, F.Cu at (199.3, -36.0)
- added R412: 1k 2%, Resistor_THT:MazdaResistor10mm, F.Cu at (38.3, -88.2)
- added R413: 36K, Resistor_THT:MazdaResistor10mm, F.Cu at (11.1, -71.4)
- added R414: 1k, Resistor_THT:MazdaResistor10mm, F.Cu at (199.3, -33.2)
- added R462: 10k, Resistor_THT:MazdaResistor10mm, F.Cu at (24.7, -82.6)
- added R471: 4.7k, Resistor_THT:MazdaResistor10mm, F.Cu at (11.1, -68.6)
- added R543: 4.7k, Resistor_THT:MazdaResistor10mm, F.Cu at (24.7, -79.8)
- added R562: 30K, Resistor_THT:MazdaResistor10mm, F.Cu at (38.3, -85.4)
- added R563: 18k, Resistor_THT:MazdaResistor10mm, F.Cu at (24.7, -77.0)
- added R603: 300R, Resistor_THT:MazdaResistor10mm, F.Cu at (11.1, -65.8)
- added R711: 300R, Resistor_THT:MazdaResistor10mm, F.Cu at (38.3, -71.4)
- added R721: 300R, Resistor_THT:MazdaResistor10mm, F.Cu at (24.7, -74.2)
- added R752: 300R, Resistor_THT:MazdaResistor10mm, F.Cu at (11.1, -63.0)
- added R762: 300R, Resistor_THT:MazdaResistor10mm, F.Cu at (11.1, -60.2)
- added R803: 4.7k, Resistor_THT:MazdaResistor10mm, F.Cu at (51.9, -88.2)
- added R804: 2.2k, Resistor_THT:MazdaResistor10mm, F.Cu at (24.7, -71.4)
- added R807: 4.7k, Resistor_THT:MazdaResistor10mm, F.Cu at (24.7, -68.6)
- added R811: 300R, Resistor_THT:MazdaResistor10mm, F.Cu at (38.3, -82.6)
- added R821: empty, Resistor_THT:MazdaResistor10mm, F.Cu at (24.7, -65.8)
- added R831: empty, Resistor_THT:MazdaResistor10mm, F.Cu at (38.3, -79.8)
- added R841: 300R, Resistor_THT:MazdaResistor10mm, F.Cu at (51.9, -85.4)
- added R851: empty, Resistor_THT:MazdaResistor10mm, F.Cu at (38.3, -77.0)
- added R912: 4.7k, Resistor_THT:MazdaResistor10mm, F.Cu at (24.7, -63.0)
- added R913: 330R, Resistor_THT:MazdaResistor10mm, F.Cu at (24.7, -60.2)
- added R922: 300R, Resistor_THT:MazdaResistor10mm, F.Cu at (38.3, -74.2)
- added R923: 330R, Resistor_THT:MazdaResistor10mm, F.Cu at (11.1, -88.2)
- C205, C452: value 47nf -> 100nf
- moved C205 103.5 mm to (38.8, -68.2)
- renumbered R521 to R520

Commit message: resistors
Parts:
- removed Empty1: BC557, Package_TO_SOT_THT:TO-92_Inline
- removed T831, T851, T861: Empty, Package_TO_SOT_THT:TO-92_Inline
- added R001: empty, ProjektMazda:MazdaResistor15mm, F.Cu at (274.4, -43.7)
- added R503: 680R, ProjektMazda:MazdaResistor12mm, F.Cu at (292.2, -71.1)
- added R723: 47R 1W, ProjektMazda:MazdaResistor15mm, F.Cu at (273.8, -71.1)
- added R754: 2.2R (m 2.8R) 1W, ProjektMazda:MazdaResistor15mm, F.Cu at (273.8, -68.3)
- added R764: 2.2R (m 2.8R) 1W, ProjektMazda:MazdaResistor15mm, F.Cu at (273.8, -65.5)
- added R802: 361R 1W, ProjektMazda:MazdaResistor15mm, F.Cu at (273.8, -62.7)
- added R842: 3.9R (m 4.8R) 1W, ProjektMazda:MazdaResistor15mm, F.Cu at (273.8, -59.9)
- added R852: empty, ProjektMazda:MazdaResistor15mm, F.Cu at (273.8, -57.1)
- added R924: empty, ProjektMazda:MazdaResistor15mm, F.Cu at (273.8, -54.3)
- added T751: CE1A3Q, Package_TO_SOT_THT:TO-126-3_Vertical, F.Cu at (120.5, -87.3)
- added T761: CE1A3Q, Package_TO_SOT_THT:TO-126-3_Vertical, F.Cu at (120.0, -77.8)
- added T812: CE1A3Q, Package_TO_SOT_THT:TO-126-3_Vertical, F.Cu at (131.4, -87.2)
- added T842: CE1A3Q, Package_TO_SOT_THT:TO-126-3_Vertical, F.Cu at (142.2, -77.3)
- R713: renamed from R503; value 680R -> 47R 1W; footprint ProjektMazda:MazdaResistor12mm -> ProjektMazda:MazdaResistor15mm
- R822, R832: footprint ProjektMazda:R17mm -> ProjektMazda:MazdaResistor15mm
- T822: value empty -> CE1A3Q (empty); footprint Package_TO_SOT_THT:MazdaTo126 -> Package_TO_SOT_THT:TO-126-3_Vertical
- T832: value Empty -> CE1A3Q (empty); footprint Package_TO_SOT_THT:MazdaTo126 -> Package_TO_SOT_THT:TO-126-3_Vertical
- T852: value empty -> CE1A3Q (empty); footprint Package_TO_SOT_THT:TO-220-3_Vertical -> Package_TO_SOT_THT:TO-126-3_Vertical
- moved T832 187.2 mm to (141.3, -87.2), turned to 0 degrees
- moved T822 177.4 mm to (131.0, -77.6), turned to 0 degrees
- moved T852 89.8 mm to (151.5, -87.1)
Connections:
- R712 pad 2: Net-(R712-Pad2) -> Net-(R711-Pad2)

Commit message: almost all elements
Parts:
- added C002: 33uf35Velec, ProjektMazda:C_Radial_D6mm_P4mm, F.Cu at (-22.2, -29.2)
- added C004: 33uf35Velec, ProjektMazda:C_Radial_D6mm_P4mm, F.Cu at (-12.1, -29.2)
- added C007: 220uf10Velec, ProjektMazda:C_Radial_D7mm_P5mm, F.Cu at (-24.2, 12.8)
- added C801: 47uf35Velec, ProjektMazda:C_Radial_D7mm_P5mm, F.Cu at (-25.7, 28.0)
- added Q802: C945, ProjektMazda:TO-92_Japan, F.Cu at (-6.53, 32.2)
- added T211: RN1006, ProjektMazda:TO-92_Japan, F.Cu at (-13.0, 38.0)
- added T711: 2CS2001, ProjektMazda:TO-92_Japan, F.Cu at (-20.9, 40.1)
- added T721: 2CS2001, ProjektMazda:TO-92_Japan, F.Cu at (-20.9, 45.9)
- added T801: 2CS2001, ProjektMazda:TO-92_Japan, F.Cu at (-38.5, 79.7)
- added T803: 2CS4065, ProjektMazda:2sc4065, F.Cu at (-9.20, 48.3)
- added T811: 2CS2001, ProjektMazda:TO-92_Japan, F.Cu at (-13.0, 32.2)
- added T821: Empty, ProjektMazda:TO-92_Japan, F.Cu at (-20.9, 51.7)
- added T831: Empty, ProjektMazda:TO-92_Japan, F.Cu at (-6.53, 38.0)
- added T841: 2CS2001, ProjektMazda:TO-92_Japan, F.Cu at (-0.02, 32.2)
- added T851: Empty, ProjektMazda:TO-92_Japan, F.Cu at (6.49, 32.2)
- added T861: Empty, ProjektMazda:TO-92_Japan, F.Cu at (13.0, 32.2)
- added T911: RN1006, ProjektMazda:TO-92_Japan, F.Cu at (-0.02, 38.0)
- added T921: RN1006, ProjektMazda:TO-92_Japan, F.Cu at (6.49, 38.0)
- J1: value Mazda_02x11 -> Conn_02x13_Odd_Even-MazdaProjekt_big; footprint ProjektMazda:EcuConnector22pin -> ProjektMazda:EcuConnector26pin
- J2: value Conn_02x13_Odd_Even -> Conn_02x11_Top_Bottom_Shielded-MazdaProjekt_big; footprint ProjektMazda:EcuConnector26pin -> ProjektMazda:EcuConnector22pin
- moved J1 39.5 mm to (85.5, 71.5)
- moved J2 37.9 mm to (79.2, 109.6)
- renumbered R001 to R1
Connections:
- R712 pad 2: Net-(R711-Pad2) -> Net-(R712-Pad2)
Routing:
- net Net-(J2-Pad2T): track 68.9 -> 0.00 mm
- net Net-(J2-Pad2Y): track 27.9 -> 0.00 mm
- net Net-(J2-Pad2W): track 6.99 -> 0.00 mm
- net Net-(J2-Pad2S): track 5.93 -> 0.00 mm

Commit message: caps and res
Parts:
- added C006: 3.3uF 16V, ProjektMazda:capacitorPolarisedMazda6mmTantalum, F.Cu at (295.9, -20.0)
- added C008: 3.3uF 16V, ProjektMazda:capacitorPolarisedMazda6mmTantalum, F.Cu at (277.7, -6.21)
- added C101: 1nF (102) 100V, ProjektMazda:capacitorTantalumMazda6mm, F.Cu at (296.2, -7.65)
- added C201: 3,3nF (332) 100V, ProjektMazda:capacitorTantalumMazda6mm, F.Cu at (299.8, -10.9)
- added C202: 3,3nF (332) 100V, ProjektMazda:capacitorTantalumMazda6mm, F.Cu at (300.4, -14.1)
- added C203: 3,3nF (332) 100V, ProjektMazda:capacitorTantalumMazda6mm, F.Cu at (296.2, -4.21)
- added C204: 1nF (102) 100V, ProjektMazda:capacitorTantalumMazda6mm, F.Cu at (304.5, -20.8)
- added C501: C_Array_7, ProjektMazda:C_array_7, F.Cu at (324.9, 36.7)
- added C502: C_Array_7, ProjektMazda:C_array_7, F.Cu at (324.9, 40.5)
- added C604: 3.3uF 16V, ProjektMazda:capacitorPolarisedMazda6mmTantalum, F.Cu at (277.7, -2.36)
- added C605: 3.3uF 16V, ProjektMazda:capacitorPolarisedMazda6mmTantalum, F.Cu at (291.8, -14.5)
- added C711: 680fF 100V, ProjektMazda:Capacitor_13mm_7m_rect_2_pin, F.Cu at (280.8, -12.9)
- added C721: 680fF 100V, ProjektMazda:Capacitor_17mm_7m_rect_3_pin, F.Cu at (280.8, -21.2)
- added J201: Connected, ProjektMazda:jumper-10E_short, F.Cu at (290.8, -4.52)
- added J601: Connected, jumper:jumper-10E, F.Cu at (298.5, -23.9)
- added R601: R_Network08_US_mazda, Resistor_THT:R_Array_SIP9, F.Cu at (205.6, -75.6)
- added R602: R_Network08_US_mazda, Resistor_THT:R_Array_SIP9, F.Cu at (205.6, -71.3)
- added R814: empty, ProjektMazda:MazdaResistor7mm, F.Cu at (306.4, -23.9)
- added R823: 4.7K, ProjektMazda:MazdaResistor7mm, F.Cu at (285.8, -7.36)
- added R833: 4.7K, ProjektMazda:MazdaResistor7mm, F.Cu at (289.4, -11.8)
- added R843: empty, ProjektMazda:MazdaResistor7mm, F.Cu at (299.9, -17.3)

Commit message: almost all elements
Parts:
- added D005: 6.2B1, ProjektMazda:diode_zener_mazda, F.Cu at (302.5, 98.9)
- added IC101: uPC177C, 40xx:40xx-DIL14, F.Cu at (333.9, -45.5)
- added IC602: TC4071BP_2, 40xx:40xx-DIL14, F.Cu at (333.9, -34.2)
- added IC603: TC4069UPB_2, 40xx:40xx-DIL14, F.Cu at (351.8, -45.5)
- R601, R602: footprint Resistor_THT:R_Array_SIP9 -> ProjektMazda:R_Array_SIP9_resistors

Commit message: 99%
Parts:
- added D2: about 27v 5W, ProjektMazda:diode_zener_mazda_big, F.Cu at (311.5, 80.9)
- added D211: Not sure propably zener, Diode_THT:DiodaMazda, F.Cu at (306.1, 91.7)
- added X601: Crystal, Crystal:Crystal_HC18-U_Vertical, F.Cu at (326.1, 59.7)
- renumbered C002 to C2, C004 to C4, C006 to C6, C007 to C7, C008 to C8, D005 to D5
