File: KiCadProject/079721-2351/079721-2351.kicad_pcb (KiCad board)
At the start: 2 copper layers, 218 parts, among them IC101 uPC177C, IC602 TC4071BP_2, IC603 TC4069UPB_2, J1 Conn_02x13_Odd_Even-MazdaProj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, J2 Conn_02x11_Top_Bottom_Shielde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, J201 Connected, J601 Connected, J711 Empty, Q802 C945, T211 RN1006, T711 2CS2001, T721 2CS2001, T751 CE1A3Q, T761 CE1A3Q, T801 2CS2001, T803 2CS4065, T811 2CS2001, T812 CE1A3Q, T821 Empty, T822 CE1A3Q (empty), T831 Empty, T832 CE1A3Q (empty), T841 2CS2001, T842 CE1A3Q, T851 Empty, T852 CE1A3Q (empty), T861 Empty, T911 RN1006, T921 RN1006, X601 Crystal

Commit message: all elements
Parts:
- added T001: 2SB1015B, ProjektMazda:TO-220-3_Vertical_Mazda, F.Cu at (-20.7, 105.7)
- added T712: 2SD1415, ProjektMazda:TO-220-3_Vertical_Mazda, F.Cu at (-20.7, 111.7)
- added T722: 2SD1415, ProjektMazda:TO-220-3_Vertical_Mazda, F.Cu at (-9.15, 105.7)
Changed lines of the file:
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@@
     (tracks 0)
     (zones 0)
-    (modules 218)
-    (nets 563)
+    (modules 221)
+    (nets 572)
   )
   (page A4)
@@
   (net 561 "Net-(X601-Pad2)")
   (net 562 "Net-(X601-Pad1)")
+  (net 563 "Net-(T001-Pad3)")
+  (net 564 "Net-(T001-Pad2)")
+  (net 565 "Net-(T001-Pad1)")
+  (net 566 "Net-(T712-Pad3)")
+  (net 567 "Net-(T712-Pad2)")
+  (net 568 "Net-(T712-Pad1)")
+  (net 569 "Net-(T722-Pad3)")
+  (net 570 "Net-(T722-Pad2)")
+  (net 571 "Net-(T722-Pad1)")
   (net_class Default "To jest domyślna klasa połączeń."
     (clearance 0.2)
@@
     (add_net "Net-(R924-Pad1)")
     (add_net "Net-(R924-Pad2)")
+    (add_net "Net-(T001-Pad1)")
+    (add_net "Net-(T001-Pad2)")
+    (add_net "Net-(T001-Pad3)")
     (add_net "Net-(T211-Pad1)")
     (add_net "Net-(T211-Pad2)")
@@
     (add_net "Net-(T711-Pad2)")
     (add_net "Net-(T711-Pad3)")
+    (add_net "Net-(T712-Pad1)")
+    (add_net "Net-(T712-Pad2)")
+    (add_net "Net-(T712-Pad3)")
     (add_net "Net-(T721-Pad1)")
     (add_net "Net-(T721-Pad2)")
     (add_net "Net-(T721-Pad3)")
+    (add_net "Net-(T722-Pad1)")
+    (add_net "Net-(T722-Pad2)")
+    (add_net "Net-(T722-Pad3)")
     (add_net "Net-(T751-Pad1)")
     (add_net "Net-(T751-Pad2)")
@@
     (add_net "Net-(c861-Pad2)")
   )
+  (module ProjektMazda:TO-220-3_Vertical_Mazda (layer F.Cu)
+    (at -9.15 105.7)
+    (descr "TO-220-3, Vertical, RM 2.54mm, see https://www.vishay.com/docs/66542/to-220-1.pdf")
+    (tags "TO-220-3 Vertical RM 2.54mm")
+    (fp_text reference T722 (at 2.3114 -3.0734) (layer F.SilkS)
+      (effects (font (size 1 1) (thickness 0.15)))
+    )
+    (fp_text value 2SD1415 (at 2.667 4.6228) (layer F.Fab)
+      (effects (font (size 1 1) (thickness 0.15)))
+    )
+    (fp_line (start 7.5438 -1.6452) (end 7.5438 -2.667) (layer F.Fab) (width 0.1))
+    (fp_line (start 7.6454 -2.667) (end 7.6454 -1.6256) (layer F.SilkS) (width 0.12))
+    (fp_line (start -0.1524 -1.651) (end -0.1524 -1.0668) (layer F.SilkS) (width 0.12))
+    (fp_line (start 2.54 -1.651) (end 2.54 1.4224) (layer F.Fab) (width 0.1))
+    (fp_line (start -2.4384 -1.6452) (end -2.4384 -2.667) (layer F.Fab) (width 0.1))
+    (fp_line (start 7.5616 -1.651) (end -2.4384 -1.651) (layer F.Fab) (width 0.1))
+    (fp_line (start -0.1524 -1.651) (end -0.1524 -0.381) (layer F.Fab) (width 0.1))
+    (fp_line (start 5.3086 -1.651) (end 5.3086 -0.381) (layer F.Fab) (width 0.1))
+    (fp_line (start -2.5908 -2.6924) (end -2.5908 -1.651) (layer F.SilkS) (width 0.12))
+    (fp_line (start -2.5946 -1.651) (end 7.6454 -1.651) (layer F.SilkS) (width 0.12))
+    (fp_line (start 2.54 -1.6256) (end 2.54 1.2192) (layer F.SilkS) (width 0.12))
+    (fp_line (start 5.3086 -1.651) (end 5.3086 -1.0668) (layer F.SilkS) (width 0.12))
+    (pad 1 thru_hole circle (at -0.2032 0) (size 2 2) (drill 1.1) (layers *.Cu *.Mask)
+      (net 571 "Net-(T722-Pad1)"))
+    (pad 2 thru_hole circle (at 2.54 2.4) (size 2 2) (drill 1.1) (layers *.Cu *.Mask)
+      (net 570 "Net-(T722-Pad2)"))
+    (pad 3 thru_hole circle (at 5.2832 0) (size 2 2) (drill 1.1) (layers *.Cu *.Mask)
+      (net 569 "Net-(T722-Pad3)"))
+    (model ${KISYS3DMOD}/Package_TO_SOT_THT.3dshapes/TO-220-3_Vertical.wrl
+      (at (xyz 0 0 0))
+      (scale (xyz 1 1 1))
+      (rotate (xyz 0 0 0))
+    )
+  )
+  (module ProjektMazda:TO-220-3_Vertical_Mazda (layer F.Cu)
+    (at -20.7 111.66)
+    (descr "TO-220-3, Vertical, RM 2.54mm, see https://www.vishay.com/docs/66542/to-220-1.pdf")
+    (tags "TO-220-3 Vertical RM 2.54mm")
+    (fp_text reference T712 (at 2.3114 -3.0734) (layer F.SilkS)
+      (effects (font (size 1 1) (thickness 0.15)))
+    )
+    (fp_text value 2SD1415 (at 2.667 4.6228) (layer F.Fab)
+      (effects (font (size 1 1) (thickness 0.15)))
+    )
+    (fp_line (start 7.5438 -1.6452) (end 7.5438 -2.667) (layer F.Fab) (width 0.1))
+    (fp_line (start 7.6454 -2.667) (end 7.6454 -1.6256) (layer F.SilkS) (width 0.12))
+    (fp_line (start -0.1524 -1.651) (end -0.1524 -1.0668) (layer F.SilkS) (width 0.12))
+    (fp_line (start 2.54 -1.651) (end 2.54 1.4224) (layer F.Fab) (width 0.1))
+    (fp_line (start -2.4384 -1.6452) (end -2.4384 -2.667) (layer F.Fab) (width 0.1))
+    (fp_line (start 7.5616 -1.651) (end -2.4384 -1.651) (layer F.Fab) (width 0.1))
+    (fp_line (start -0.1524 -1.651) (end -0.1524 -0.381) (layer F.Fab) (width 0.1))
+    (fp_line (start 5.3086 -1.651) (end 5.3086 -0.381) (layer F.Fab) (width 0.1))
+    (fp_line (start -2.5908 -2.6924) (end -2.5908 -1.651) (layer F.SilkS) (width 0.12))
+    (fp_line (start -2.5946 -1.651) (end 7.6454 -1.651) (layer F.SilkS) (width 0.12))
+    (fp_line (start 2.54 -1.6256) (end 2.54 1.2192) (layer F.SilkS) (width 0.12))
+    (fp_line (start 5.3086 -1.651) (end 5.3086 -1.0668) (layer F.SilkS) (width 0.12))
+    (pad 1 thru_hole circle (at -0.2032 0) (size 2 2) (drill 1.1) (layers *.Cu *.Mask)
+      (net 568 "Net-(T712-Pad1)"))
+    (pad 2 thru_hole circle (at 2.54 2.4) (size 2 2) (drill 1.1) (layers *.Cu *.Mask)
+      (net 567 "Net-(T712-Pad2)"))
+    (pad 3 thru_hole circle (at 5.2832 0) (size 2 2) (drill 1.1) (layers *.Cu *.Mask)
+      (net 566 "Net-(T712-Pad3)"))
+    (model ${KISYS3DMOD}/Package_TO_SOT_THT.3dshapes/TO-220-3_Vertical.wrl
+      (at (xyz 0 0 0))
+      (scale (xyz 1 1 1))
+      (rotate (xyz 0 0 0))
+    )
+  )
+  (module ProjektMazda:TO-220-3_Vertical_Mazda (layer F.Cu)
+    (at -20.7 105.7)
+    (descr "TO-220-3, Vertical, RM 2.54mm, see https://www.vishay.com/docs/66542/to-220-1.pdf")
+    (tags "TO-220-3 Vertical RM 2.54mm")
+    (fp_text reference T001 (at 2.3114 -3.0734) (layer F.SilkS)
+      (effects (font (size 1 1) (thickness 0.15)))
+    )
+    (fp_text value 2SB1015B (at 2.667 4.6228) (layer F.Fab)
+      (effects (font (size 1 1) (thickness 0.15)))
+    )
+    (fp_line (start 7.5438 -1.6452) (end 7.5438 -2.667) (layer F.Fab) (width 0.1))
+    (fp_line (start 7.6454 -2.667) (end 7.6454 -1.6256) (layer F.SilkS) (width 0.12))
+    (fp_line (start -0.1524 -1.651) (end -0.1524 -1.0668) (layer F.SilkS) (width 0.12))
+    (fp_line (start 2.54 -1.651) (end 2.54 1.4224) (layer F.Fab) (width 0.1))
+    (fp_line (start -2.4384 -1.6452) (end -2.4384 -2.667) (layer F.Fab) (width 0.1))
+    (fp_line (start 7.5616 -1.651) (end -2.4384 -1.651) (layer F.Fab) (width 0.1))
+    (fp_line (start -0.1524 -1.651) (end -0.1524 -0.381) (layer F.Fab) (width 0.1))
+    (fp_line (start 5.3086 -1.651) (end 5.3086 -0.381) (layer F.Fab) (width 0.1))
+    (fp_line (start -2.5908 -2.6924) (end -2.5908 -1.651) (layer F.SilkS) (width 0.12))
+    (fp_line (start -2.5946 -1.651) (end 7.6454 -1.651) (layer F.SilkS) (width 0.12))
+    (fp_line (start 2.54 -1.6256) (end 2.54 1.2192) (layer F.SilkS) (width 0.12))
+    (fp_line (start 5.3086 -1.651) (end 5.3086 -1.0668) (layer F.SilkS) (width 0.12))
+    (pad 1 thru_hole circle (at -0.2032 0) (size 2 2) (drill 1.1) (layers *.Cu *.Mask)
+      (net 565 "Net-(T001-Pad1)"))
+    (pad 2 thru_hole circle (at 2.54 2.4) (size 2 2) (drill 1.1) (layers *.Cu *.Mask)
+      (net 564 "Net-(T001-Pad2)"))
+    (pad 3 thru_hole circle (at 5.2832 0) (size 2 2) (drill 1.1) (layers *.Cu *.Mask)
+      (net 563 "Net-(T001-Pad3)"))
+    (model ${KISYS3DMOD}/Package_TO_SOT_THT.3dshapes/TO-220-3_Vertical.wrl
+      (at (xyz 0 0 0))
+      (scale (xyz 1 1 1))
+      (rotate (xyz 0 0 0))
+    )
+  )
   (module Crystal:Crystal_HC18-U_Vertical (layer F.Cu)
